File: Prototype_Payload_Controller/Payload_Controller_EM.kicad_sch (KiCad schematic)
At the start: 4 parts

Commit message: Updated For Review
Changed lines of the file:
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@@
+	)
+	(junction
+		(at 318.77 111.76)
+		(diameter 0)
+		(color 0 0 0 0)
+	)
+	(junction
+		(at 322.58 107.95)
+		(diameter 0)
+		(color 0 0 0 0)
+	)
+	(junction
+		(at 322.58 111.76)
+		(diameter 0)
+		(color 0 0 0 0)
 	)
 	(junction
@@
 	(wire
 		(pts
+			(xy 322.58 111.76) (xy 322.58 114.3)
+		)
+		(stroke
+			(width 0)
+			(type default)
+		)
+	)
+	(wire
+		(pts
 			(xy 299.72 107.95) (xy 318.77 107.95)
 		)
@@
 	(wire
 		(pts
+			(xy 322.58 107.95) (xy 322.58 111.76)
+		)
+		(stroke
+			(width 0)
+			(type default)
+		)
+	)
+	(wire
+		(pts
 			(xy 232.918 147.32) (xy 252.73 147.32)
 		)
@@
 	(wire
 		(pts
+			(xy 318.77 111.76) (xy 322.58 111.76)
+		)
+		(stroke
+			(width 0)
+			(type default)
+		)
+	)
+	(wire
+		(pts
 			(xy 313.69 104.14) (xy 327.152 104.14)
 		)
@@
 		)
 	)
+	(wire
+		(pts
+			(xy 322.58 114.3) (xy 318.77 114.3)
+		)
+		(stroke
+			(width 0)
+			(type default)
+		)
+	)
 	(bus
 		(pts
@@
 	(wire
 		(pts
-			(xy 318.77 107.95) (xy 327.152 107.95)
+			(xy 318.77 107.95) (xy 322.58 107.95)
+		)
+		(stroke
+			(width 0)
+			(type default)
+		)
+	)
+	(wire
+		(pts
+			(xy 318.77 111.76) (xy 318.77 114.3)
 		)
 		(stroke
@@
 		)
 	)
+	(wire
+		(pts
+			(xy 318.77 107.95) (xy 318.77 111.76)
+		)
+		(stroke
+			(width 0)
+			(type default)
+		)
+	)
 	(bus
 		(pts
@@
 		)
 		(stroke
+			(width 0)
+			(type default)
+		)
+	)
+	(wire
+		(pts
+			(xy 322.58 107.95) (xy 327.152 107.95)
+		)
+		(stroke
