File: RM-VT01A_Breakout_Board_Prototype/RM-VT01A_Breakout_Board.kicad_pcb (KiCad board)
At the start: 4 copper layers, 43.8 x 38.7 mm, 15 parts, among them J1 Conn_Coaxial, J2 Conn_01x06

Commit message: Updated For Review
Parts:
- J2: footprint Connector_Hirose:Hirose_DF11-6DP-2DSA_2x03_P2.00mm_Vertical -> PinHeader:PinHeader_2x03_P2.00mm_Vertical
Changed lines of the file:
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@@
 			(outputformat 1)
 			(mirror no)
-			(drillshape 1)
+			(drillshape 0)
 			(scaleselection 1)
 			(outputdirectory "")
@@
 		(sheetname "/")
 		(sheetfile "RM-VT01A_Breakout_Board.kicad_sch")
-		(attr through_hole)
+		(attr through_hole exclude_from_pos_files exclude_from_bom)
 		(fp_circle
 			(center 0 0)
@@
 			)
 		)
+		(property "LCSC" "C3172376"
+			(at 0 0 0)
+			(layer "F.SilkS")
+			(hide yes)
+			(effects
+				(font
+					(size 1.27 1.27)
+					(thickness 0.15)
+				)
+			)
+		)
 		(property ki_fp_filters "*BNC* *SMA* *SMB* *SMC* *Cinch* *LEMO* *UMRF* *MCX* *U.FL*")
 		(sheetname "/")
@@
 			)
 		)
+		(property "LCSC" "C1691"
+			(at 0 0 0)
+			(layer "F.SilkS")
+			(hide yes)
+			(effects
+				(font
+					(size 1.27 1.27)
+					(thickness 0.15)
+				)
+			)
+		)
 		(property ki_fp_filters "C_*")
 		(sheetname "/")
@@
 		(sheetname "/")
 		(sheetfile "RM-VT01A_Breakout_Board.kicad_sch")
-		(attr through_hole)
+		(attr through_hole exclude_from_pos_files exclude_from_bom)
 		(fp_circle
 			(center 0 0)
@@
 		(sheetname "/")
 		(sheetfile "RM-VT01A_Breakout_Board.kicad_sch")
-		(attr through_hole)
+		(attr through_hole exclude_from_pos_files exclude_from_bom)
 		(fp_circle
 			(center 0 0)
@@
 		(sheetname "/")
 		(sheetfile "RM-VT01A_Breakout_Board.kicad_sch")
-		(attr through_hole)
+		(attr through_hole exclude_from_pos_files exclude_from_bom)
 		(fp_circle
 			(center 0 0)
@@
 		(sheetname "/")
 		(sheetfile "RM-VT01A_Breakout_Board.kicad_sch")
-		(attr smd)
+		(attr smd exclude_from_pos_files exclude_from_bom)
 		(fp_line
 			(start -6.75 -12)
@@
 		(sheetname "/")
 		(sheetfile "RM-VT01A_Breakout_Board.kicad_sch")
-		(attr through_hole)
+		(attr through_hole exclude_from_pos_files exclude_from_bom)
 		(fp_circle
 			(center 0 0)
@@
 		(embedded_fonts no)
 	)
-	(footprint "Connector_Hirose:Hirose_DF11-6DP-2DSA_2x03_P2.00mm_Vertical"
+	(footprint "PinHeader:PinHeader_2x03_P2.00mm_Vertical"
 		(layer "F.Cu")
 		(at 128.0668 78.391 -90)
@@
 		(tags "connector Hirose DF11 vertical")
 		(property "Reference" "J2"
-			(at -3.2258 1.0602 0)
+			(at 2 -2.7 270)
 			(layer "F.SilkS")
 			(effects
@@
 		)
 		(property "Value" "Conn_01x06"
-			(at 2 4.7 90)
+			(at 2 4.7 270)
 			(layer "F.Fab")
 			(effects
@@
 		(property "Datasheet" ""
 			(at 0 0 270)
-			(unlocked yes)
 			(layer "F.Fab")
 			(hide yes)
@@
 		(property "Description" "Generic connector, single row, 01x06, script generated (kicad-library-utils/schlib/autogen/connector/)"
 			(at 0 0 270)
-			(unlocked yes)
 			(layer "F.Fab")
 			(hide yes)
@@
 		(sheetname "/")
 		(sheetfile "RM-VT01A_Breakout_Board.kicad_sch")
-		(attr through_hole)
+		(attr through_hole exclude_from_pos_files exclude_from_bom)
 		(fp_line
 			(start -2.1 3.6)
@@
 		)
 		(fp_text user "${REFERENCE}"
-			(at 2 2.8 90)
+			(at 2 2.8 270)
 			(layer "F.Fab")
 			(effects
@@
 		)
 		(embedded_fonts no)
-		(model "${KICAD9_3DMODEL_DIR}/Connector_Hirose.3dshapes/Hirose_DF11-6DP-2DSA_2x03_P2.00mm_Vertical.wrl"
+		(model "${KICAD9_3DMODEL_DIR}/Connector_Hirose.3dshapes/Hirose_DF11-6DP-2DSA_2x03_P2.00mm_Vertical.step"
 			(offset
 				(xyz 0 0 0)
@@
 			)
 		)
+		(model "C:/Users/perso/Downloads/PARTserver22026091206525459527728d0b6156e/TMM-103-01-L-D.stp"
+			(offset
+				(xyz 2 -1 1.5)
+			)
+			(scale
+				(xyz 1 1 1)
+			)
+			(rotate
+				(xyz 90 -0 -0)
+			)
+		)
+		(model "${KIPRJMOD}/PinHeader.pretty/TMM-103-01-L-D.stp"
+			(offset
+				(xyz 2 -1.5 -3)
+			)
+			(scale
+				(xyz 1 1 1)
+			)
+			(rotate
+				(xyz -90 -0 -0)
+			)
+		)
