File: RM-VT01A_Breakout_Board_Prototype/RM-VT01A_Breakout_Board.kicad_sch (KiCad schematic)
At the start: 13 parts, among them J1 Conn_Coaxial, J2 Conn_01x06

Commit message: Updated For Review
Parts:
- J2: footprint Connector_Hirose:Hirose_DF11-6DP-2DSA_2x03_P2.00mm_Vertical -> PinHeader:PinHeader_2x03_P2.00mm_Vertical
Changed lines of the file:
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@@
 			)
 		)
-		(property "Footprint" "Connector_Hirose:Hirose_DF11-6DP-2DSA_2x03_P2.00mm_Vertical"
+		(property "Footprint" "PinHeader:PinHeader_2x03_P2.00mm_Vertical"
 			(at 44.45 91.44 0)
 			(effects
